Commit message: chapt6完结，实现gazebo世界构建和机器人导入与控制

File: chapt6/chapt6_ws/src/fishbot_description/urdf/first_robot.xacro (robot description, xacro)
@@ -1,6 +1,7 @@
 <?xml version="1.0"?>
-<robot name="first_robot">
-    <!-- 机器人的身体部分 -->
-    <link name="base_link">
+<robot xmlns:xacro="http://www.ros.org/wiki/xacro" name="first_robot">
+    <xacro:macro name="base_link" params="length radius">
+        <!-- 机器人的身体部分 -->
+        <link name="base_link">
             <!-- 部件外观描述 -->
             <visual>
@@ -10,5 +11,5 @@
                 <geometry>
                     <!-- 圆柱体,半径0.10 高度0.12 -->
-                    <cylinder radius="0.10" length="0.12"/>
+                    <cylinder radius="${radius}" length="${length}"/>
                 </geometry>
                 <!-- 材质颜色 -->
@@ -17,7 +18,9 @@
                 </material>
             </visual>
-    </link>
-    <!-- 机器人的IMU部件，惯性测量传感器 -->
-    <link name="imu_link">
+        </link>
+    </xacro:macro>
+    <xacro:macro name="imu_link" params="imu_name xyz">
+        <!-- 机器人的IMU部件，惯性测量传感器 -->
+        <link name="${imu_name}_link">
             <!-- 部件外观描述 -->
             <visual>
@@ -33,10 +36,14 @@
                 </material>
             </visual>
-    </link>
+        </link>
     <!-- 机器人的关节，用于组合机器人的部件 -->
-    <joint name="imu_joint" type="fixed">
-        <origin xyz="0.0 0.0 0.03" rpy="0.0 0.0 0.0"/>
+    <joint name="${imu_name}_joint" type="fixed">
+        <origin xyz="${xyz}" rpy="0.0 0.0 0.0"/>
         <parent link="base_link"/>
-        <child link="imu_link"/>
+        <child link="${imu_name}_link"/>
     </joint>
+    </xacro:macro>
+    <xacro:base_link length="0.12" radius="0.1"/>
+    <xacro:imu_link imu_name="imu_up" xyz="0.0 0.0 0.03"/>
+    <xacro:imu_link imu_name="imu_down" xyz="0.0 0.0 -0.03"/>
 </robot>

File: chapt6/chapt6_ws/src/fishbot_description/urdf/fishbot/sensor/camera.urdf.xacro (robot description, xacro)
@@ -1,6 +1,8 @@
 <?xml version="1.0"?>
-<robot name="first_robot">
-    <!-- 机器人的身体部分 -->
-    <link name="base_link">
+<robot xmlns:xacro="http://www.ros.org/wiki/xacro">
+<xacro:include filename="$(find fishbot_description)/urdf/fishbot/common_inertia.xacro"/>
+    <xacro:macro name="camera_xacro" params="xyz">
+        <!-- 机器人的IMU部件，惯性测量传感器 -->
+        <link name="camera_link">
             <!-- 部件外观描述 -->
             <visual>
@@ -9,22 +11,5 @@
                 <!-- 几何形状 -->
                 <geometry>
-                    <!-- 圆柱体,半径0.10 高度0.12 -->
-                    <cylinder radius="0.10" length="0.12"/>
-                </geometry>
-                <!-- 材质颜色 -->
-                <material name="white">
-                    <color rgba="1.0 1.0 1.0 0.5"/>
-                </material>
-            </visual>
-    </link>
-    <!-- 机器人的IMU部件，惯性测量传感器 -->
-    <link name="imu_link">
-            <!-- 部件外观描述 -->
-            <visual>
-                <!-- 沿着自己几何中心的偏移和旋转量 -->
-                <origin xyz="0.0 0.0 0.0" rpy="0.0 0.0 0.0"/>
-                <!-- 几何形状 -->
-                <geometry>
-                    <box size="0.02 0.02 0.02"/>
+                    <box size="0.02 0.10 0.02"/>
                 </geometry>
                 <!-- 材质颜色 -->
@@ -33,10 +18,24 @@
                 </material>
             </visual>
-    </link>
+            <collision>
+                <!-- 沿着自己几何中心的偏移和旋转量 -->
+                <origin xyz="0.0 0.0 0.0" rpy="0.0 0.0 0.0"/>
+                <!-- 几何形状 -->
+                <geometry>
+                    <box size="0.02 0.10 0.02"/>
+                </geometry>
+                <!-- 材质颜色 -->
+                <material name="black">
+                    <color rgba="0.0 0.0 0.0 0.5"/>
+                </material>
+            </collision>
+            <xacro:box_inertia m="0.1" w="0.02" h="0.10" d="0.02" />
+        </link>
     <!-- 机器人的关节，用于组合机器人的部件 -->
-    <joint name="imu_joint" type="fixed">
-        <origin xyz="0.0 0.0 0.03" rpy="0.0 0.0 0.0"/>
+    <joint name="camera_joint" type="fixed">
+        <origin xyz="${xyz}" rpy="0.0 0.0 0.0"/>
         <parent link="base_link"/>
-        <child link="imu_link"/>
+        <child link="camera_link"/>
     </joint>
+    </xacro:macro>
 </robot>

File: chapt6/chapt6_ws/src/fishbot_description/urdf/fishbot/sensor/imu.urdf.xacro (robot description, xacro)
@@ -1,23 +1,8 @@
 <?xml version="1.0"?>
-<robot name="first_robot">
-    <!-- 机器人的身体部分 -->
-    <link name="base_link">
-            <!-- 部件外观描述 -->
-            <visual>
-                <!-- 沿着自己几何中心的偏移和旋转量 -->
-                <origin xyz="0.0 0.0 0.0" rpy="0.0 0.0 0.0"/>
-                <!-- 几何形状 -->
-                <geometry>
-                    <!-- 圆柱体,半径0.10 高度0.12 -->
-                    <cylinder radius="0.10" length="0.12"/>
-                </geometry>
-                <!-- 材质颜色 -->
-                <material name="white">
-                    <color rgba="1.0 1.0 1.0 0.5"/>
-                </material>
-            </visual>
-    </link>
-    <!-- 机器人的IMU部件，惯性测量传感器 -->
-    <link name="imu_link">
+<robot xmlns:xacro="http://www.ros.org/wiki/xacro">
+<xacro:include filename="$(find fishbot_description)/urdf/fishbot/common_inertia.xacro"/>
+    <xacro:macro name="imu_xacro" params="xyz">
+        <!-- 机器人的IMU部件，惯性测量传感器 -->
+        <link name="imu_link">
             <!-- 部件外观描述 -->
             <visual>
@@ -33,10 +18,24 @@
                 </material>
             </visual>
-    </link>
+            <collision>
+                <!-- 沿着自己几何中心的偏移和旋转量 -->
+                <origin xyz="0.0 0.0 0.0" rpy="0.0 0.0 0.0"/>
+                <!-- 几何形状 -->
+                <geometry>
+                    <box size="0.02 0.02 0.02"/>
+                </geometry>
+                <!-- 材质颜色 -->
+                <material name="black">
+                    <color rgba="0.0 0.0 0.0 0.5"/>
+                </material>
+            </collision>
+            <xacro:box_inertia m="0.05" w="0.02" h="0.02" d="0.02" />
+        </link>
     <!-- 机器人的关节，用于组合机器人的部件 -->
     <joint name="imu_joint" type="fixed">
-        <origin xyz="0.0 0.0 0.03" rpy="0.0 0.0 0.0"/>
+        <origin xyz="${xyz}" rpy="0.0 0.0 0.0"/>
         <parent link="base_link"/>
         <child link="imu_link"/>
     </joint>
+    </xacro:macro>
 </robot>
