Commit message: 5.22nav2

File: chapt6/chapt6_ws/src/fishbot_description/urdf/fishbot/actuator/caster.urdf.xacro (robot description, xacro)
@@ -32,11 +32,17 @@
         </link>
     <!-- 机器人的关节，用于组合机器人的部件 -->
-    <joint name="${caster_name}_joint" type="fixed">
-        <origin xyz="${xyz}" rpy="0.0 0.0 0.0"/>
-        <parent link="base_link"/>
-        <child link="${caster_name}_link"/>
-        <axis xyz="0.0 1.0 0.0"/>
-    </joint>
-    <xacro:sphere_inertia m="0.05" r="0.016" />
+        <joint name="${caster_name}_joint" type="fixed">
+            <origin xyz="${xyz}" rpy="0.0 0.0 0.0"/>
+            <parent link="base_link"/>
+            <child link="${caster_name}_link"/>
+            <axis xyz="0.0 1.0 0.0"/>
+        </joint>
+        <gazebo reference="${caster_name}_link">
+            <mu1 value="0.0"/>
+            <mu2 value="0.0"/>
+            <kp value="1000000000.0"/>
+            <kd value="1.0"/>
+        </gazebo>
+        <xacro:sphere_inertia m="0.05" r="0.016" />
     </xacro:macro>
 </robot>

File: chapt6/chapt6_ws/src/fishbot_description/urdf/fishbot/actuator/wheel.urdf.xacro (robot description, xacro)
@@ -30,13 +30,19 @@
                 </material>
             </collision>
-            <xacro:cylinder_inertia m="0.05" r="${radius}" h="${length}" />
+            <xacro:cylinder_inertia m="0.05" r="0.032" h="0.04" />
         </link>
-    <!-- 机器人的关节，用于组合机器人的部件 -->
-    <joint name="${wheel_name}_joint" type="continuous">
-        <origin xyz="${xyz}" rpy="0.0 0.0 0.0"/>
-        <parent link="base_link"/>
-        <child link="${wheel_name}_link"/>
-        <axis xyz="0.0 1.0 0.0"/>
-    </joint>
+        <!-- 机器人的关节，用于组合机器人的部件 -->
+        <joint name="${wheel_name}_joint" type="continuous">
+            <origin xyz="${xyz}" rpy="0.0 0.0 0.0"/>
+            <parent link="base_link"/>
+            <child link="${wheel_name}_link"/>
+            <axis xyz="0.0 1.0 0.0"/>
+        </joint>
+        <gazebo reference="${wheel_name}_link">
+            <mu1 value="20.0"/>
+            <mu2 value="20.0"/>
+            <kp value="1000000000.0"/>
+            <kd value="1.0"/>
+        </gazebo>
     </xacro:macro>
 </robot>

File: chapt6/chapt6_ws/src/fishbot_description/urdf/fishbot/fishbot.urdf.xacro (robot description, xacro)
@@ -10,11 +10,18 @@
     <xacro:include filename="$(find fishbot_description)/urdf/fishbot/actuator/wheel.urdf.xacro"/>
     <xacro:include filename="$(find fishbot_description)/urdf/fishbot/actuator/caster.urdf.xacro"/>
+     <!-- 插件 -->
+    <xacro:include filename="$(find fishbot_description)/urdf/fishbot/plugins/gazebo_control_plugin.xacro"/>
+    <xacro:include filename="$(find fishbot_description)/urdf/fishbot/plugins/gazebo_sensor_plugin.xacro"/>
+    <xacro:include filename="$(find fishbot_description)/urdf/fishbot/fishbot.ros2_control.xacro"/>
     <xacro:base_xacro length="0.12" radius="0.10"/>
     <xacro:imu_xacro xyz="0.0 0.0 0.02"/>
     <xacro:camera_xacro xyz="0.10 0.0 0.075"/>
-    <xacro:laser_xacro xyz="0.10 0.0 0.10"/>
+    <xacro:laser_xacro xyz="0.0 0.0 0.10"/>
     <xacro:wheel_xacro wheel_name="left_wheel" xyz="0.0 0.10 -0.06"/>
     <xacro:wheel_xacro wheel_name="right_wheel" xyz="0.0 -0.10 -0.06"/>
     <xacro:caster_xacro caster_name="front_caster" xyz="0.08 0.0 -0.076"/>
     <xacro:caster_xacro caster_name="back_caster" xyz="-0.08 0.0 -0.076"/>
+    <!-- <xacro:gazebo_control_plugin /> -->
+    <xacro:gazebo_sensor_plugin />
+    <xacro:fishbot_ros2_control />
 </robot>

File: chapt6/chapt6_ws/src/fishbot_description/urdf/fishbot/sensor/camera.urdf.xacro (robot description, xacro)
@@ -32,10 +32,17 @@
             <xacro:box_inertia m="0.1" w="0.02" h="0.10" d="0.02" />
         </link>
+        <link name="camera_optical_link">
+        </link>
     <!-- 机器人的关节，用于组合机器人的部件 -->
-    <joint name="camera_joint" type="fixed">
-        <origin xyz="${xyz}" rpy="0.0 0.0 0.0"/>
-        <parent link="base_link"/>
-        <child link="camera_link"/>
-    </joint>
+        <joint name="camera_joint" type="fixed">
+            <origin xyz="${xyz}" rpy="0.0 0.0 0.0"/>
+            <parent link="base_link"/>
+            <child link="camera_link"/>
+        </joint>
+        <joint name="camera_optical_joint" type="fixed">
+            <origin xyz="0 0 0" rpy="${-pi/2} 0.0 0.0"/>
+            <parent link="camera_link"/>
+            <child link="camera_optical_link"/>
+        </joint>
     </xacro:macro>
 </robot>

File: chapt6/chapt6_ws/src/fishbot_description/urdf/fishbot/sensor/laser.urdf.xacro (robot description, xacro)
@@ -72,4 +72,10 @@
             <child link="laser_cylinder_link"/>
         </joint>
+        <gazebo reference="laser_cylinder_link">
+            <material>Gazebo/Black</material>
+        </gazebo>
+        <gazebo reference="laser_link">
+            <material>Gazebo/Black</material>
+        </gazebo>
     </xacro:macro>
 </robot>
