Commit message: chapt7结束

File: chapt7/chapt7_ws/src/fishbot_description/urdf/first_robot.urdf (robot description, URDF)
Before this commit: robot first_robot, 2 links, 1 joints
Joints:
- joint imu_joint: origin xyz=0.0 0.0 0.03 rpy=0.0 0.0 0.0 -> xyz=0 0 0.03 rpy=0 0 0

File: chapt7/chapt7_ws/src/fishbot_description/urdf/fishbot/actuator/caster.urdf.xacro (robot description, xacro)
@@ -1,48 +1,39 @@
 <?xml version="1.0"?>
 <robot xmlns:xacro="http://www.ros.org/wiki/xacro">
-<xacro:include filename="$(find fishbot_description)/urdf/fishbot/common_inertia.xacro"/>
+   <xacro:include filename="$(find fishbot_description)/urdf/fishbot/common_inertia.xacro" />
     <xacro:macro name="caster_xacro" params="caster_name xyz">
-        <!-- 机器人的IMU部件，惯性测量传感器 -->
-        <link name="${caster_name}_link">
-            <!-- 部件外观描述 -->
+        <link name="${caster_name}_caster_link">
             <visual>
-                <!-- 沿着自己几何中心的偏移和旋转量 -->
-                <origin xyz="0.0 0.0 0.0" rpy="1.57079 0.0 0.0"/>
-                <!-- 几何形状 -->
+                <origin xyz="0 0 0" rpy="0 0 0" />
                 <geometry>
-                    <sphere radius="0.016"/>
+                    <sphere radius="0.016" />
                 </geometry>
-                <!-- 材质颜色 -->
-                <material name="yellow">
-                    <color rgba="1.0 1.0 0.0 1.0"/>
+                <material name="black">
+                    <color rgba="0.0 0.0 0.0 0.8"/>
                 </material>
             </visual>
             <collision>
-                <!-- 沿着自己几何中心的偏移和旋转量 -->
-                <origin xyz="0.0 0.0 0.0" rpy="1.57079 0.0 0.0"/>
-                <!-- 几何形状 -->
+                <origin xyz="0 0 0" rpy="0 0 0" />
                 <geometry>
-                    <sphere radius="0.016"/>
+                    <sphere radius="0.016" />
                 </geometry>
-                <!-- 材质颜色 -->
-                <material name="yellow">
-                    <color rgba="1.0 1.0 0.0 1.0"/>
+                <material name="black">
+                    <color rgba="0.0 0.0 0.0 0.8"/>
                 </material>
             </collision>
+            <xacro:sphere_inertia m="0.01" r="0.016" />
         </link>
-    <!-- 机器人的关节，用于组合机器人的部件 -->
-        <joint name="${caster_name}_joint" type="fixed">
-            <origin xyz="${xyz}" rpy="0.0 0.0 0.0"/>
-            <parent link="base_link"/>
-            <child link="${caster_name}_link"/>
-            <axis xyz="0.0 1.0 0.0"/>
+        <gazebo reference="${caster_name}_caster_link">
+            <mu1 value="0.0" />
+            <mu2 value="0.0" />
+            <kp value="1000000000.0" />
+            <kd value="1.0" />
+        </gazebo>
+        <joint name="${caster_name}_caster_joint" type="fixed">
+            <parent link="base_link" />
+            <child link="${caster_name}_caster_link" />
+            <origin xyz="${xyz}" />
+            <axis xyz="0 0 0" />
         </joint>
-        <gazebo reference="${caster_name}_link">
-            <mu1 value="0.0"/>
-            <mu2 value="0.0"/>
-            <kp value="1000000000.0"/>
-            <kd value="1.0"/>
-        </gazebo>
-        <xacro:sphere_inertia m="0.05" r="0.016" />
     </xacro:macro>
 </robot>

File: chapt7/chapt7_ws/src/fishbot_description/urdf/fishbot/actuator/wheel.urdf.xacro (robot description, xacro)
@@ -1,48 +1,39 @@
 <?xml version="1.0"?>
 <robot xmlns:xacro="http://www.ros.org/wiki/xacro">
-<xacro:include filename="$(find fishbot_description)/urdf/fishbot/common_inertia.xacro"/>
+   <xacro:include filename="$(find fishbot_description)/urdf/fishbot/common_inertia.xacro" />
     <xacro:macro name="wheel_xacro" params="wheel_name xyz">
-        <!-- 机器人的IMU部件，惯性测量传感器 -->
-        <link name="${wheel_name}_link">
-            <!-- 部件外观描述 -->
+        <link name="${wheel_name}_wheel_link">
             <visual>
-                <!-- 沿着自己几何中心的偏移和旋转量 -->
-                <origin xyz="0.0 0.0 0.0" rpy="1.57079 0.0 0.0"/>
-                <!-- 几何形状 -->
+                <origin xyz="0 0 0" rpy="1.57079 0 0" />
                 <geometry>
-                    <cylinder radius="0.032" length="0.04"/>
+                    <cylinder length="0.04" radius="0.032" />
                 </geometry>
-                <!-- 材质颜色 -->
-                <material name="yellow">
-                    <color rgba="1.0 1.0 0.0 1.0"/>
+                <material name="black">
+                    <color rgba="0.0 0.0 0.0 0.8"/>
                 </material>
             </visual>
             <collision>
-                <!-- 沿着自己几何中心的偏移和旋转量 -->
-                <origin xyz="0.0 0.0 0.0" rpy="1.57079 0.0 0.0"/>
-                <!-- 几何形状 -->
+                <origin xyz="0 0 0" rpy="1.57079 0 0" />
                 <geometry>
-                    <cylinder radius="0.032" length="0.04"/>
+                    <cylinder length="0.04" radius="0.032" />
                 </geometry>
-                <!-- 材质颜色 -->
-                <material name="yellow">
-                    <color rgba="1.0 1.0 0.0 1.0"/>
+                <material name="black">
+                    <color rgba="0.0 0.0 0.0 0.8"/>
                 </material>
             </collision>
-            <xacro:cylinder_inertia m="0.05" r="0.032" h="0.04" />
+            <xacro:cylinder_inertia m="0.1" h="0.04" r="0.032"/>
         </link>
-        <!-- 机器人的关节，用于组合机器人的部件 -->
-        <joint name="${wheel_name}_joint" type="continuous">
-            <origin xyz="${xyz}" rpy="0.0 0.0 0.0"/>
-            <parent link="base_link"/>
-            <child link="${wheel_name}_link"/>
-            <axis xyz="0.0 1.0 0.0"/>
+        <gazebo reference="${wheel_name}_wheel_link">
+            <mu1 value="20.0" />
+            <mu2 value="20.0" />
+            <kp value="1000000000.0" />
+            <kd value="1.0" />
+        </gazebo>
+        <joint name="${wheel_name}_wheel_joint" type="continuous">
+            <parent link="base_link" />
+            <child link="${wheel_name}_wheel_link" />
+            <origin xyz="${xyz}" />
+            <axis xyz="0 1 0" />
         </joint>
-        <gazebo reference="${wheel_name}_link">
-            <mu1 value="20.0"/>
-            <mu2 value="20.0"/>
-            <kp value="1000000000.0"/>
-            <kd value="1.0"/>
-        </gazebo>
     </xacro:macro>
 </robot>

File: chapt7/chapt7_ws/src/fishbot_description/urdf/fishbot/base.urdf.xacro (robot description, xacro)
@@ -1,43 +1,33 @@
 <?xml version="1.0"?>
 <robot xmlns:xacro="http://www.ros.org/wiki/xacro">
-    <xacro:include filename="$(find fishbot_description)/urdf/fishbot/common_inertia.xacro"/>
+   <xacro:include filename="$(find fishbot_description)/urdf/fishbot/common_inertia.xacro" />
     <xacro:macro name="base_xacro" params="length radius">
-        <link name="base_footprint" />
-        <!-- 机器人的身体部分 -->
+     <link name="base_footprint" />
+        <joint name="base_joint" type="fixed">
+            <parent link="base_footprint" />
+            <child link="base_link" />
+            <origin xyz="0.0 0.0 ${length/2.0+0.032-0.001}" rpy="0 0 0" />
+        </joint>
         <link name="base_link">
-            <!-- 部件外观描述 -->
             <visual>
-                <!-- 沿着自己几何中心的偏移和旋转量 -->
-                <origin xyz="0.0 0.0 0.0" rpy="0.0 0.0 0.0"/>
-                <!-- 几何形状 -->
+                <origin xyz="0 0 0.0" rpy="0 0 0" />
                 <geometry>
-                    <!-- 圆柱体,半径0.10 高度0.12 -->
-                    <cylinder radius="${radius}" length="${length}"/>
+                    <cylinder length="${length}" radius="${length}" />
                 </geometry>
-                <!-- 材质颜色 -->
-                <material name="white">
-                    <color rgba="1.0 1.0 1.0 0.5"/>
+                <material name="blue">
+                    <color rgba="0.1 0.1 1.0 0.5"/>
                 </material>
             </visual>
             <collision>
-                <!-- 沿着自己几何中心的偏移和旋转量 -->
-                <origin xyz="0.0 0.0 0.0" rpy="0.0 0.0 0.0"/>
-                <!-- 几何形状 -->
+                <origin xyz="0 0 0.0" rpy="0 0 0" />
                 <geometry>
-                    <!-- 圆柱体,半径0.10 高度0.12 -->
-                    <cylinder radius="${radius}" length="${length}"/>
+                    <cylinder length="${length}" radius="${length}" />
                 </geometry>
-                <!-- 材质颜色 -->
-                <material name="white">
-                    <color rgba="1.0 1.0 1.0 0.5"/>
+                <material name="blue">
+                    <color rgba="0.1 0.1 1.0 0.5"/>
                 </material>
             </collision>
-            <xacro:cylinder_inertia m="1.0" r="${radius}" h="${length}" />
+            <xacro:cylinder_inertia m="1.0" r="${radius}" h="${length}"/>
         </link>
-        <joint name="joint_name" type="fixed">
-            <origin xyz="0.0 0.0 ${length/2.0+0.032-0.001}" rpy="0.0 0.0 0.0"/>
-            <parent link="base_footprint"/>
-            <child link="base_link"/>
-        </joint>
     </xacro:macro>
 </robot>

File: chapt7/chapt7_ws/src/fishbot_description/urdf/fishbot/fishbot.ros2_control.xacro (robot description, xacro)
@@ -2,5 +2,5 @@
 <robot xmlns:xacro="http://www.ros.org/wiki/xacro">
     <xacro:macro name="fishbot_ros2_control">
-        <ros2_control name="FishBotGazeboSystem" type="system">
+    <ros2_control name="FishBotGazeboSystem" type="system">
             <hardware>
                 <plugin>gazebo_ros2_control/GazeboSystem</plugin>
@@ -37,6 +37,6 @@
             <parameters>$(find fishbot_description)/config/fishbot_ros2_controller.yaml</parameters>
             <ros>
+                <remapping>/fishbot_diff_drive_controller/cmd_vel_unstamped:=/cmd_vel</remapping>
                 <remapping>/fishbot_diff_drive_controller/odom:=/odom</remapping>
-                <remapping>/fishbot_diff_drive_controller/cmd_vel_unstamped:=/cmd_vel</remapping>
             </ros>
         </plugin>

File: chapt7/chapt7_ws/src/fishbot_description/urdf/fishbot/fishbot.urdf.xacro (robot description, xacro)
@@ -1,27 +1,28 @@
 <?xml version="1.0"?>
-<robot xmlns:xacro="http://www.ros.org/wiki/xacro" name="fish_bot">
-    <!-- 基础部分 -->
-    <xacro:include filename="$(find fishbot_description)/urdf/fishbot/base.urdf.xacro"/>
-    <!-- 传感器部分 -->
-    <xacro:include filename="$(find fishbot_description)/urdf/fishbot/sensor/imu.urdf.xacro"/>
-    <xacro:include filename="$(find fishbot_description)/urdf/fishbot/sensor/camera.urdf.xacro"/>
-    <xacro:include filename="$(find fishbot_description)/urdf/fishbot/sensor/laser.urdf.xacro"/>
-    <!-- 执行器部分 -->
-    <xacro:include filename="$(find fishbot_description)/urdf/fishbot/actuator/wheel.urdf.xacro"/>
-    <xacro:include filename="$(find fishbot_description)/urdf/fishbot/actuator/caster.urdf.xacro"/>
-     <!-- 插件 -->
-    <xacro:include filename="$(find fishbot_description)/urdf/fishbot/plugins/gazebo_control_plugin.xacro"/>
-    <xacro:include filename="$(find fishbot_description)/urdf/fishbot/plugins/gazebo_sensor_plugin.xacro"/>
-    <xacro:include filename="$(find fishbot_description)/urdf/fishbot/fishbot.ros2_control.xacro"/>
-    <xacro:base_xacro length="0.12" radius="0.10"/>
-    <xacro:imu_xacro xyz="0.0 0.0 0.02"/>
-    <xacro:camera_xacro xyz="0.10 0.0 0.075"/>
-    <xacro:laser_xacro xyz="0.0 0.0 0.10"/>
-    <xacro:wheel_xacro wheel_name="left_wheel" xyz="0.0 0.10 -0.06"/>
-    <xacro:wheel_xacro wheel_name="right_wheel" xyz="0.0 -0.10 -0.06"/>
-    <xacro:caster_xacro caster_name="front_caster" xyz="0.08 0.0 -0.076"/>
-    <xacro:caster_xacro caster_name="back_caster" xyz="-0.08 0.0 -0.076"/>
+<robot xmlns:xacro="http://www.ros.org/wiki/xacro" name="fishbot">
+    <xacro:include filename="$(find fishbot_description)/urdf/fishbot/base.urdf.xacro" />
+    <!-- 传感器组件 -->
+    <xacro:include filename="$(find fishbot_description)/urdf/fishbot/sensor/imu.urdf.xacro" />
+    <xacro:include filename="$(find fishbot_description)/urdf/fishbot/sensor/laser.urdf.xacro" />
+    <xacro:include filename="$(find fishbot_description)/urdf/fishbot/sensor/camera.urdf.xacro" />
+     <!-- 执行器组件 -->
+    <xacro:include filename="$(find fishbot_description)/urdf/fishbot/actuator/wheel.urdf.xacro" />
+    <xacro:include filename="$(find fishbot_description)/urdf/fishbot/actuator/caster.urdf.xacro" />
+    <xacro:base_xacro length="0.12" radius="0.1" />
+    <!-- 传感器 -->
+    <xacro:imu_xacro xyz="0 0 0.02" />
+    <xacro:laser_xacro xyz="0 0 0.10" />
+    <xacro:camera_xacro xyz="0.10 0 0.075" />
+    <!-- 执行器主动轮+从动轮 -->
+    <xacro:wheel_xacro wheel_name="left" xyz="0 0.10 -0.06" />
+    <xacro:wheel_xacro wheel_name="right" xyz="0 -0.10 -0.06" />
+    <xacro:caster_xacro caster_name="front" xyz="0.08 0.0 -0.076" />
+    <xacro:caster_xacro caster_name="back" xyz="-0.08 0.0 -0.076" />
+    <!-- Gazebo 插件 -->
+    <xacro:include filename="$(find fishbot_description)/urdf/fishbot/plugins/gazebo_control_plugin.xacro" />
     <!-- <xacro:gazebo_control_plugin /> -->
+    <xacro:include filename="$(find fishbot_description)/urdf/fishbot/fishbot.ros2_control.xacro" />
+    <xacro:fishbot_ros2_control />
+    <xacro:include filename="$(find fishbot_description)/urdf/fishbot/plugins/gazebo_sensor_plugin.xacro" />
     <xacro:gazebo_sensor_plugin />
-    <xacro:fishbot_ros2_control />
 </robot>

File: chapt7/chapt7_ws/src/fishbot_description/urdf/fishbot/plugins/gazebo_sensor_plugin.xacro (robot description, xacro)
@@ -14,5 +14,5 @@
                 <always_on>true</always_on>
                 <visualize>false</visualize>
-                <update_rate>100</update_rate>
+                <update_rate>10</update_rate>
                 <pose>0 0 0 0 0 0</pose>
 								<!-- 激光传感器配置 -->

File: chapt7/chapt7_ws/src/fishbot_description/urdf/fishbot/sensor/camera.urdf.xacro (robot description, xacro)
@@ -1,47 +1,38 @@
 <?xml version="1.0"?>
 <robot xmlns:xacro="http://www.ros.org/wiki/xacro">
-<xacro:include filename="$(find fishbot_description)/urdf/fishbot/common_inertia.xacro"/>
+   <xacro:include filename="$(find fishbot_description)/urdf/fishbot/common_inertia.xacro" />
     <xacro:macro name="camera_xacro" params="xyz">
-        <!-- 机器人的IMU部件，惯性测量传感器 -->
+        <!-- ============相机模块================ -->
         <link name="camera_link">
-            <!-- 部件外观描述 -->
             <visual>
-                <!-- 沿着自己几何中心的偏移和旋转量 -->
-                <origin xyz="0.0 0.0 0.0" rpy="0.0 0.0 0.0"/>
-                <!-- 几何形状 -->
+                <origin xyz="0 0 0.0" rpy="0 0 0" />
                 <geometry>
-                    <box size="0.02 0.10 0.02"/>
+                    <box size="0.02 0.10 0.02" />
                 </geometry>
-                <!-- 材质颜色 -->
                 <material name="black">
-                    <color rgba="0.0 0.0 0.0 0.5"/>
+                    <color rgba="0.0 0.0 0.0 0.8"/>
                 </material>
             </visual>
             <collision>
-                <!-- 沿着自己几何中心的偏移和旋转量 -->
-                <origin xyz="0.0 0.0 0.0" rpy="0.0 0.0 0.0"/>
-                <!-- 几何形状 -->
+                <origin xyz="0 0 0.0" rpy="0 0 0" />
                 <geometry>
-                    <box size="0.02 0.10 0.02"/>
+                    <box size="0.02 0.10 0.02" />
                 </geometry>
-                <!-- 材质颜色 -->
                 <material name="black">
-                    <color rgba="0.0 0.0 0.0 0.5"/>
+                    <color rgba="0.0 0.0 0.0 0.8"/>
                 </material>
             </collision>
-            <xacro:box_inertia m="0.1" w="0.02" h="0.10" d="0.02" />
+            <xacro:box_inertia m="0.01" w="0.02" h="0.10" d="0.02" />
         </link>
-        <link name="camera_optical_link">
-        </link>
-    <!-- 机器人的关节，用于组合机器人的部件 -->
+        <link name="camera_optical_link"></link>
+        <joint name="camera_optical_joint" type="fixed">
+            <parent link="camera_link" />
+            <child link="camera_optical_link" />
+            <origin xyz="0 0 0" rpy="${-pi/2} 0 ${-pi/2}" />
+        </joint>
         <joint name="camera_joint" type="fixed">
-            <origin xyz="${xyz}" rpy="0.0 0.0 0.0"/>
-            <parent link="base_link"/>
-            <child link="camera_link"/>
-        </joint>
-        <joint name="camera_optical_joint" type="fixed">
-            <origin xyz="0 0 0" rpy="${-pi/2} 0.0 0.0"/>
-            <parent link="camera_link"/>
-            <child link="camera_optical_link"/>
+            <parent link="base_link" />
+            <child link="camera_link" />
+            <origin xyz="${xyz}" />
         </joint>
     </xacro:macro>

File: chapt7/chapt7_ws/src/fishbot_description/urdf/fishbot/sensor/imu.urdf.xacro (robot description, xacro)
@@ -1,41 +1,32 @@
 <?xml version="1.0"?>
 <robot xmlns:xacro="http://www.ros.org/wiki/xacro">
-<xacro:include filename="$(find fishbot_description)/urdf/fishbot/common_inertia.xacro"/>
+   <xacro:include filename="$(find fishbot_description)/urdf/fishbot/common_inertia.xacro" />
     <xacro:macro name="imu_xacro" params="xyz">
-        <!-- 机器人的IMU部件，惯性测量传感器 -->
         <link name="imu_link">
-            <!-- 部件外观描述 -->
             <visual>
-                <!-- 沿着自己几何中心的偏移和旋转量 -->
-                <origin xyz="0.0 0.0 0.0" rpy="0.0 0.0 0.0"/>
-                <!-- 几何形状 -->
+                <origin xyz="0 0 00" rpy="0 0 0" />
                 <geometry>
-                    <box size="0.02 0.02 0.02"/>
+                    <box size="0.02 0.02 0.02" />
                 </geometry>
-                <!-- 材质颜色 -->
                 <material name="black">
-                    <color rgba="0.0 0.0 0.0 0.5"/>
+                    <color rgba="0 0 0 0.8" />
                 </material>
             </visual>
             <collision>
-                <!-- 沿着自己几何中心的偏移和旋转量 -->
-                <origin xyz="0.0 0.0 0.0" rpy="0.0 0.0 0.0"/>
-                <!-- 几何形状 -->
+                <origin xyz="0 0 00" rpy="0 0 0" />
                 <geometry>
-                    <box size="0.02 0.02 0.02"/>
+                    <box size="0.02 0.02 0.02" />
                 </geometry>
-                <!-- 材质颜色 -->
                 <material name="black">
-                    <color rgba="0.0 0.0 0.0 0.5"/>
+                    <color rgba="0 0 0 0.8" />
                 </material>
             </collision>
-            <xacro:box_inertia m="0.05" w="0.02" h="0.02" d="0.02" />
+            <xacro:box_inertia m="0.01" w="0.02" d="0.02" h="0.02"/>
         </link>
-    <!-- 机器人的关节，用于组合机器人的部件 -->
-    <joint name="imu_joint" type="fixed">
-        <origin xyz="${xyz}" rpy="0.0 0.0 0.0"/>
-        <parent link="base_link"/>
-        <child link="imu_link"/>
-    </joint>
+        <joint name="imu_joint" type="fixed">
+            <parent link="base_link" />
+            <child link="imu_link" />
+            <origin xyz="${xyz}" />
+        </joint>
     </xacro:macro>
 </robot>
