Commit message: chapt7结束

File: chapt7/chapt7_ws/src/fishbot_description/urdf/fishbot/sensor/laser.urdf.xacro (robot description, xacro)
@@ -1,75 +1,6 @@
 <?xml version="1.0"?>
 <robot xmlns:xacro="http://www.ros.org/wiki/xacro">
-<xacro:include filename="$(find fishbot_description)/urdf/fishbot/common_inertia.xacro"/>
+   <xacro:include filename="$(find fishbot_description)/urdf/fishbot/common_inertia.xacro" />
     <xacro:macro name="laser_xacro" params="xyz">
-        <!-- 雷达支撑杆 -->
-        <link name="laser_cylinder_link">
-            <!-- 部件外观描述 -->
-            <visual>
-                <!-- 沿着自己几何中心的偏移和旋转量 -->
-                <origin xyz="0.0 0.0 0.0" rpy="0.0 0.0 0.0"/>
-                <!-- 几何形状 -->
-                <geometry>
-                    <cylinder radius="0.01" length="0.10"/>
-                </geometry>
-                <!-- 材质颜色 -->
-                <material name="black">
-                    <color rgba="0.0 0.0 0.0 1.0"/>
-                </material>
-            </visual>
-            <collision>
-                <!-- 沿着自己几何中心的偏移和旋转量 -->
-                <origin xyz="0.0 0.0 0.0" rpy="0.0 0.0 0.0"/>
-                <!-- 几何形状 -->
-                <geometry>
-                    <cylinder radius="0.01" length="0.10"/>
-                </geometry>
-                <!-- 材质颜色 -->
-                <material name="black">
-                    <color rgba="0.0 0.0 0.0 1.0"/>
-                </material>
-            </collision>
-            <xacro:cylinder_inertia m="0.05" r="0.01" h="0.10" />
-        </link>
-        <!-- 雷达 -->
-        <link name="laser_link">
-            <!-- 部件外观描述 -->
-            <visual>
-                <!-- 沿着自己几何中心的偏移和旋转量 -->
-                <origin xyz="0.0 0.0 0.0" rpy="0.0 0.0 0.0"/>
-                <!-- 几何形状 -->
-                <geometry>
-                    <cylinder radius="0.02" length="0.02"/>
-                </geometry>
-                <!-- 材质颜色 -->
-                <material name="black">
-                    <color rgba="0.0 0.0 0.0 1.0"/>
-                </material>
-            </visual>
-            <collision>
-                <!-- 沿着自己几何中心的偏移和旋转量 -->
-                <origin xyz="0.0 0.0 0.0" rpy="0.0 0.0 0.0"/>
-                <!-- 几何形状 -->
-                <geometry>
-                    <cylinder radius="0.02" length="0.02"/>
-                </geometry>
-                <!-- 材质颜色 -->
-                <material name="black">
-                    <color rgba="0.0 0.0 0.0 1.0"/>
-                </material>
-            </collision>
-            <xacro:cylinder_inertia m="0.10" r="0.02" h="0.02" />
-        </link>
-        <!-- 机器人的关节，用于组合机器人的部件 -->
-        <joint name="laser_joint" type="fixed">
-            <origin xyz="0.0 0.0 0.05" rpy="0.0 0.0 0.0"/>
-            <parent link="laser_cylinder_link"/>
-            <child link="laser_link"/>
-        </joint>
-        <joint name="laser_cylinder_joint" type="fixed">
-            <origin xyz="${xyz}" rpy="0.0 0.0 0.0"/>
-            <parent link="base_link"/>
-            <child link="laser_cylinder_link"/>
-        </joint>
         <gazebo reference="laser_cylinder_link">
             <material>Gazebo/Black</material>
@@ -78,4 +9,58 @@
             <material>Gazebo/Black</material>
         </gazebo>
+        <!-- ============雷达支撑杆================ -->
+        <link name="laser_cylinder_link">
+            <visual>
+                <origin xyz="0 0 0" rpy="0 0 0" />
+                <geometry>
+                    <cylinder length="0.10" radius="0.01" />
+                </geometry>
+                <material name="black">
+                    <color rgba="0.0 0.0 0.0 0.8" />
+                </material>
+            </visual>
+            <collision>
+                <origin xyz="0 0 0" rpy="0 0 0" />
+                <geometry>
+                    <cylinder length="0.10" radius="0.01" />
+                </geometry>
+                <material name="black">
+                    <color rgba="0.0 0.0 0.0 0.8" />
+                </material>
+            </collision>
+            <xacro:cylinder_inertia m="0.01" r="0.01" h="0.10" />
+        </link>
+        <joint name="laser_cylinder_joint" type="fixed">
+            <parent link="base_link" />
+            <child link="laser_cylinder_link" />
+            <origin xyz="${xyz}" />
+        </joint>
+        <!-- ============雷达================ -->
+        <link name="laser_link">
+            <visual>
+                <origin xyz="0 0 0" rpy="0 0 0" />
+                <geometry>
+                    <cylinder length="0.02" radius="0.02" />
+                </geometry>
+                <material name="black">
+                    <color rgba="0.0 0.0 0.0 0.8" />
+                </material>
+            </visual>
+            <collision>
+                <origin xyz="0 0 0" rpy="0 0 0" />
+                <geometry>
+                    <cylinder length="0.02" radius="0.02" />
+                </geometry>
+                <material name="black">
+                    <color rgba="0.0 0.0 0.0 0.8" />
+                </material>
+            </collision>
+            <xacro:cylinder_inertia m="0.03" r="0.02" h="0.02" />
+        </link>
+        <joint name="laser_joint" type="fixed">
+            <parent link="laser_cylinder_link" />
+            <child link="laser_link" />
+            <origin xyz="0 0 0.05" />
+        </joint>
     </xacro:macro>
 </robot>
